File: SuperSamFPGA.kicad_sch (KiCad schematic)
At the start: 102 parts, among them J1 DataBus, J2 Video, J3 AddressBus, J4 ControlOut, J5 ControlIn, J6 JTAG, SW1 Tactile, U10 TXS0108EPW, U11 TXS0104EPW, U12 TXS0104EPW, U13 NCP1529A, U14 NCP1529A, U15 TPS563201, U2 XC7A15T-CSG325, U3 IS61WV51216BLL, U4 IS61WV51216BLL, U5 MX25L6433F, U6 SN74AC17PWR, U7 SN74AC17PWR, U9 AT28BV64B-20JU, Y1 SiT8008xx-2x-xxS

Commit message: complete initial design
Parts:
- added J7: BusService, Connector_PinHeader_2.54mm:PinHeader_1x10_P2.54mm_Vertical, symbol Connector_Generic:Conn_01x10
- added J8: RomAddr, Connector_PinHeader_2.54mm:PinHeader_1x08_P2.54mm_Vertical, symbol Connector_Generic:Conn_01x08
- added U1: 74LVC573, Package_SO:TSSOP-20_4.4x6.5mm_P0.65mm, symbol 74xx:74LS373
- C1, C30, C31, C33, C34, C35, C36, C37, C41, C42, C6, C7, C9: LCSC (none) -> C1705
- C10, C11, C2, C25, C29, C3, C32, C4, C40, C43, C44, C45, C5, C8: LCSC (none) -> C1525
- C26, C27: footprint Capacitor_SMD:C_0402_1005Metric -> Capacitor_SMD:C_0805_2012Metric
- C38, C39: LCSC (none) -> C1555
- D1: LCSC (none) -> C51933298
- D2: LCSC (none) -> C2286
- L1, L2: LCSC (none) -> C86090
- L3: LCSC (none) -> C703091
- R1, R2, R3, R4, R5: LCSC (none) -> C105871
- R10, R8, R9: LCSC C4109 -> C60490
- R11, R6, R7: LCSC (none) -> C11702
- R12: LCSC (none) -> C23162
- R13: LCSC (none) -> C191123
- R14, R17: LCSC (none) -> C93947
- R15: LCSC (none) -> C25798
- R16, R18: LCSC (none) -> C60491
- R19: LCSC (none) -> C25779
- SW1: LCSC (none) -> C49108628
- U13, U14: LCSC (none) -> C49375212
- U15: LCSC (none) -> C116592
- U2: LCSC (none) -> C1551978
- U3: value IS61WV51216BLL -> IS61WV51216BLL-10TLI; DigiKey (none) -> 706-1107-ND; LCSC C397874 -> C6968505
- U4: LCSC C397874 -> C6968505
- U5: LCSC (none) -> C706695
- Y1: LCSC (none) -> C2901579
Connections:
- net +3V3: now also U1.20 (VCC)
- net A0: now also U2.B11 (IO_L4N_T0_15); no longer U2.E13 (IO_L12P_T1_MRCC_15)
- net A1: now also U2.C12 (IO_L6N_T0_VREF_15); no longer U2.D13 (IO_L11P_T1_SRCC_15)
- net A11: now also U2.B15 (IO_L9N_T1_DQS_AD3N_15); no longer U2.C16 (IO_L16P_T2_A28_15)
- net A12: now also U2.D15 (IO_L13N_T2_MRCC_15); no longer U2.B16 (IO_L15P_T2_DQS_15)
- net A13: now also U2.B16 (IO_L15P_T2_DQS_15); no longer U2.C17 (IO_L18P_T2_A24_15)
- net A2: now also U2.A12 (IO_L7N_T1_AD2N_15); no longer U2.A13 (IO_L8P_T1_AD10P_15)
- net A3: now also U2.B12 (IO_L7P_T1_AD2P_15); no longer U2.C13 (IO_L11N_T1_SRCC_15)
- net A5: now also U2.C13 (IO_L11N_T1_SRCC_15); no longer U2.C14 (IO_L9P_T1_DQS_AD3P_15)
- net A6: now also U2.A13 (IO_L8P_T1_AD10P_15); no longer U2.A14 (IO_L8N_T1_AD10N_15)
- net A7: now also U2.A14 (IO_L8N_T1_AD10N_15); no longer U2.B14 (IO_L10P_T1_AD11P_15)
- net A8: now also U2.B14 (IO_L10P_T1_AD11P_15); no longer U2.D15 (IO_L13N_T2_MRCC_15)
- net A9: now also U2.C14 (IO_L9P_T1_DQS_AD3P_15); no longer U2.B15 (IO_L9N_T1_DQS_AD3N_15)
- net CSS: now also U2.C16 (IO_L16P_T2_A28_15); no longer U2.C18 (IO_L18N_T2_A23_15)
- net E: now also U2.E18 (IO_L24N_T3_RS0_15); no longer U2.F17 (IO_L24P_T3_RS1_15)
- net GM1: now also U2.D18 (IO_L17N_T2_A25_15); no longer U2.E17 (IO_L17P_T2_A26_15)
- net GM2: now also U2.E17 (IO_L17P_T2_A26_15); no longer U2.E18 (IO_L24N_T3_RS0_15)
- net GND: now also U2.D11 (IO_L6P_T0_15), J7.10 (Pin_10), U1.1 (OE), U1.10 (GND), U1.18 (D7)
- net RD0: now also U1.8 (D3); no longer U9.7 (A4)
- net RD1: now also U1.7 (D2); no longer U9.6 (A5)
- net RD2: now also U1.4 (D1); no longer U9.5 (A6)
- net RD3: now also U1.3 (D0); no longer U9.4 (A7)
- net RD4: now also U1.17 (D6); no longer U9.29 (A8)
- net RD5: now also U1.14 (D5); no longer U9.28 (A9)
- net RD6: now also U1.13 (D4); no longer U9.24 (A10)
- net R/~{W}: now also U2.D16 (IO_L14N_T2_SRCC_15); no longer U2.E15 (IO_L13P_T2_MRCC_15)
- net S0: now also U2.F17 (IO_L24P_T3_RS1_15); no longer U2.G15 (IO_L21P_T3_DQS_15)
- net ~{A}/G: now also U2.C18 (IO_L18N_T2_A23_15); no longer U2.D18 (IO_L17N_T2_A25_15)
- net ~{RST}: now also U2.C17 (IO_L18P_T2_A24_15); no longer U2.D16 (IO_L14N_T2_SRCC_15)
- net RZ16: now reaches U2.G14 (IO_L22P_T3_A17_15)
- net RZ16: now also J8.4 (Pin_4)
- net RZ18: now reaches U2.H14 (IO_25_15)
- net RZ18: now also J8.6 (Pin_6)
- net RZ14: now reaches U2.H16 (IO_L20P_T3_A20_15)
- net RZ14: now also J8.2 (Pin_2)
- net RZ17: now reaches U2.H17 (IO_L23P_T3_FOE_B_15)
- net RZ17: now also J8.5 (Pin_5)
- net RZ15: now reaches U2.H18 (IO_L23N_T3_FWE_B_15)
- net RZ15: now also J8.3 (Pin_3)
- net ~{RWE}: now reaches U2.J18 (IO_L3P_T0_DQS_PUDC_B_14)
- net ~{RWE}: now also J8.7 (Pin_7)
- net ~{ROE}: now reaches U2.K18 (IO_L3N_T0_DQS_EMCCLK_14)
- net ~{ROE}: now also J8.8 (Pin_8)
- net ~{NMI}: now reaches U2.L18 (IO_L4N_T0_D05_14)
- net ~{NMI}: now also J7.1 (Pin_1)
- net ~{IRQ}: now reaches U2.M15 (IO_L6N_T0_D08_VREF_14)
- net ~{IRQ}: now also J7.3 (Pin_3)
- net ~{FIRQ}: now reaches U2.M16 (IO_L7P_T1_D09_14)
- net ~{FIRQ}: now also J7.2 (Pin_2)
- net BA: now reaches U2.N14 (IO_L8N_T1_D12_14)
- net BA: now also J7.5 (Pin_5)
- net BS: now reaches U2.N16 (IO_L9P_T1_DQS_14)
- net BS: now also J7.4 (Pin_4)
- net HALT: now reaches U2.P15 (IO_L11P_T1_SRCC_14)
- net HALT: now also J7.6 (Pin_6)
- net LIC: now reaches U2.P16 (IO_L11N_T1_SRCC_14)
- net LIC: now also J7.8 (Pin_8)
- net TSC: now reaches U2.R15 (IO_L12N_T1_MRCC_14)
- net TSC: now also J7.7 (Pin_7)
- net AVMA: now reaches U2.R16 (IO_L14P_T2_SRCC_14)
- net AVMA: now also J7.9 (Pin_9)
- net RLE: now reaches U2.V4 (IO_L18N_T2_34)
- net RLE: now also U1.11 (LE)
- new net CC0: U1.9 (O3), U9.7 (A4)
- new net CC1: U1.6 (O2), U9.6 (A5)
- new net CC2: U1.5 (O1), U9.5 (A6)
- new net CC3: U1.2 (O0), U9.4 (A7)
- new net CC4: U1.16 (O6), U9.29 (A8)
- new net CC5: U1.15 (O5), U9.28 (A9)
- new net CC6: U1.12 (O4), U9.24 (A10)
- new net RZ13: J8.1 (Pin_1), U2.G15 (IO_L21P_T3_DQS_15)
- no-connect marks 26 -> 27
Other:
- moved on the sheet: C1, C10, C11, C12, C14, C15, C17, C18, C2, C20, C21, C22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

Commit message: implement alternative sram
Parts:
- removed U3: IS61WV51216BLL-10TLI, Package_SO:TSOP-II-44_10.16x18.41mm_P0.8mm, symbol Library:IS61WV51216BLL
- removed U4: IS61WV51216BLL, Package_SO:TSOP-II-44_10.16x18.41mm_P0.8mm, symbol Library:IS61WV51216BLL
- added C23: 100nF, Capacitor_SMD:C_0402_1005Metric, symbol Device:C
- added U8: CY7C10612G30-10ZSXI, PCM_Package_SO_AKL:TSOP-II-54_22.2x10.16mm_P0.8mm, symbol Library:CY7C10612G30-10ZSXI
Connections:
- net +3V3: now also C23.1, U8.14 (VCC), U8.2 (VCC), U8.23 (VCC), U8.29 (VCC), U8.50 (VCC)
- net GND: now also C23.2, U8.26 (VSS), U8.32 (VSS), U8.41 (VSS), U8.42 (*OE), U8.5 (VSS), U8.53 (VSS)
- net RD0: now also U8.25 (I/O2), U8.4 (I/O14)
- net RD1: now also U8.24 (I/O1), U8.3 (I/O13)
- net RD2: now also U8.1 (I/O12), U8.22 (I/O0)
- net RD3: now also U8.27 (I/O3), U8.6 (I/O15)
- net RD4: now also U8.28 (I/O4), U8.49 (I/O8)
- net RD5: now also U8.33 (I/O7), U8.54 (I/O11)
- net RD6: now also U8.31 (I/O6), U8.52 (I/O10)
- net RD7: now also U8.30 (I/O5), U8.51 (I/O9)
- net Z0: now also U8.39 (*BLE)
- net Z1: now also U8.7 (A4)
- net Z10: now also U8.38 (A10)
- net Z11: now also U8.37 (A11)
- net Z12: now also U8.36 (A12)
- net Z13: now also U8.35 (A13)
- net Z14: now also U8.34 (A14)
- net Z15: now also U8.18 (A18)
- net Z16: now also U8.17 (A19)
- net Z17: now also U8.11 (A0)
- net Z18: now also U8.10 (A1)
- net Z19: now also U8.48 (A5)
- net Z2: now also U8.8 (A3)
- net Z3: now also U8.9 (A2)
- net Z4: now also U8.21 (A15)
- net Z5: now also U8.20 (A16)
- net Z6: now also U8.47 (A6)
- net Z7: now also U8.46 (A7)
- net Z8: now also U8.45 (A8)
- net Z9: now also U8.44 (A9)
- net ~{WE}: now also U8.15 (*WE)
- net ~{Z0}: now also U8.12 (*BHE)
- net ~{CE}1 renamed ~{CE}
- net ~{CE}: now also U8.13 (*CE)
- net ~{CE}2 renamed Z20
- net Z20: now also U8.19 (A17)
Other:
- moved on the sheet: C12, C15, C21, C22

Commit message: switch to single chip dac
Parts:
- removed R10, R8, R9: 470R, PCM_Resistor_SMD_AKL:R_0402_1005Metric, symbol Device:R_Small
- removed RN1, RN2, RN3: 33R, PCM_Resistor_SMD_AKL:R_Array_Convex_4x0402, symbol PCM_Resistor_AKL:R_4x0402_Convex
- removed RN4, RN5, RN6: 470R, PCM_Resistor_SMD_AKL:R_Array_Convex_4x0402, symbol PCM_Resistor_AKL:R_4x0402_Convex
- removed RN7, RN8, RN9: 220R, PCM_Resistor_SMD_AKL:R_Array_Convex_4x0402, symbol PCM_Resistor_AKL:R_4x0402_Convex
- removed U6, U7: SN74AC17PWR, Package_SO:TSSOP-14_4.4x5mm_P0.65mm, symbol 74xx:74HC7014
- added C24, C28: 10uF, Capacitor_SMD:C_0805_2012Metric, symbol Device:C
- added C46, C47, C48, C49, C50: 100nF, Capacitor_SMD:C_0402_1005Metric, symbol Device:C
- added L4, L5: 4.7uH, Inductor_SMD:L_0805_2012Metric, symbol Device:L_Small
- added R20, R22: 2.2K, PCM_Resistor_SMD_AKL:R_0402_1005Metric, symbol Device:R_Small
- added R21: 3.8K, PCM_Resistor_SMD_AKL:R_0402_1005Metric, symbol Device:R_Small
- added U3: THS8136IPHP, Library:PHP48_4P1X4P1, symbol Library:THS8136IPHP
- C26: value 100uF -> 10uF; LCSC Part C1525 -> (none)
- C27: value 100uF -> 10uF
Connections:
- net +1V8: now also C24.1, L4.1, R20.2
- net +3V3: now also C46.1, C49.2, L5.1; no longer C18.1, C27.1
- net B0: now also U2.N4 (IO_L10N_T1_34), U3.7 (B3); no longer U2.K6 (IO_L1P_T0_34)
- net B1: now also U2.L2 (IO_L4N_T0_34), U3.8 (B2); no longer U2.J4 (IO_L2N_T0_34)
- net B2: now also U2.L3 (IO_L5N_T0_34), U3.9 (B1); no longer U2.J6 (IO_0_34)
- net B3: now also U2.L4 (IO_L5P_T0_34), U3.10 (B0); no longer U2.J5 (IO_L2P_T0_34)
- net BLUE: now also J2.6 (Pin_6), U3.45 (AB); no longer J2.2 (Pin_2)
- net Format: now also U2.M4 (IO_L10P_T1_34); no longer U2.L5 (IO_L6P_T0_34)
- net G0: now also U2.J6 (IO_0_34), U3.30 (G6); no longer U2.K2 (IO_L3P_T0_DQS_34)
- net G1: now also U2.J5 (IO_L2P_T0_34), U3.29 (G7); no longer U2.K1 (IO_L3N_T0_DQS_34)
- net G2: now also U2.J4 (IO_L2N_T0_34), U3.28 (G8); no longer U2.K3 (IO_L4P_T0_34)
- net G3: now also U2.K6 (IO_L1P_T0_34), U3.27 (G9); no longer U2.K5 (IO_L1N_T0_34)
- net GND: now also C24.2, C28.2, C46.2, C47.2, C48.2, C50.2, R21.1, R22.1, U3.1 (B9), U3.11 (DVSS), U3.13 (R0), U3.14 (R1), U3.15 (R2), U3.16 (R3), U3.17 (R4), U3.18 (R5), U3.2 (B8), U3.3 (B7), U3.31 (G5), U3.32 (G4), U3.33 (G3), U3.34 (G2), U3.35 (G1), U3.36 (G0), U3.4 (B6), U3.42 (AVSS), U3.46 (AVSS), U3.5 (B5), U3.6 (B4), U3.EPAD
- net GREEN: now also J2.2 (Pin_2), U3.41 (AG); no longer J2.4 (Pin_4)
- net R0: now also U2.K1 (IO_L3N_T0_DQS_34), U3.19 (R6); no longer U2.L3 (IO_L5N_T0_34)
- net R1: now also U2.K2 (IO_L3P_T0_DQS_34), U3.20 (R7); no longer U2.L4 (IO_L5P_T0_34)
- net R2: now also U2.K3 (IO_L4P_T0_34), U3.21 (R8); no longer U2.L2 (IO_L4N_T0_34)
- net R3: now also U2.K5 (IO_L1N_T0_34), U3.22 (R9); no longer U2.N4 (IO_L10N_T1_34)
- net RED: now also J2.4 (Pin_4), U3.43 (AR); no longer J2.6 (Pin_6)
- new net: R21.2, U3.38 (FSAADJ)
- new net: R22.2, U3.47 (M1), U3.48 (M2)
- new net: C50.1, U3.37 (VREF)
- new net: C49.1, U3.39 (COMP)
- new net: R20.1, U3.23 (*BLANK), U3.24 (*SYNC), U3.25 (SYNC-T)
- new net AVDD: C18.1, C27.1, C48.1, L5.2, U3.40 (AVDD), U3.44 (AVDD)
- new net DVDD: C28.1, C47.1, L4.2, U3.12 (DVDD)
- new net VCLK: U2.L5 (IO_L6P_T0_34), U3.26 (CLK)
- no-connect marks 27 -> 21
Other:
- moved on the sheet: C13, C14, C15, C16, C17, C18, C19, C20, C21, C22, C23, C26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

Commit message: production ready
Parts:
- added U4: IS61WV102416BLL-10TLI, Package_SO:TSOP-I-48_18.4x12mm_P0.5mm, symbol Library:IS61WV102416BLL-10TLI
- C12, U8: now left out of the parts list
- C18: LCSC Part C1525 -> C141660
- C24, C26, C27, C28: LCSC C141660 -> C15850
- D1: LCSC C51933298 -> C2290
- R1, R2, R3, R4, R5: LCSC C105871 -> C25900
- R13: LCSC C191123 -> C25744
- R16, R18: LCSC C60491 -> C25741
- R20, R22: LCSC (none) -> C25879
- R21: LCSC (none) -> C852772
Connections:
- net +3V3: now also U4.12 (VDD), U4.36 (VDD)
- net GND: now also U4.13 (GND), U4.37 (GND), U4.44 (*OE)
- net RD0: now also U4.17 (I/O7), U4.32 (I/O8)
- net RD1: now also U4.16 (I/O6), U4.33 (I/O9)
- net RD2: now also U4.15 (I/O5), U4.34 (I/O10)
- net RD3: now also U4.14 (I/O4), U4.35 (I/O11)
- net RD4: now also U4.11 (I/O3), U4.38 (I/O12)
- net RD5: now also U4.10 (I/O2), U4.39 (I/O13)
- net RD6: now also U4.40 (I/O14), U4.9 (I/O1)
- net RD7: now also U4.41 (I/O15), U4.8 (I/O0)
- net Z0: now also U4.42 (*LB)
- net Z1: now also U4.1 (A4)
- net Z10: now also U4.23 (A16)
- net Z11: now also U4.24 (A15)
- net Z12: now also U4.48 (A5)
- net Z13: now also U4.47 (A6)
- net Z14: now also U4.46 (A7)
- net Z15: now also U4.45 (A8)
- net Z16: now also U4.27 (A12)
- net Z17: now also U4.26 (A13)
- net Z18: now also U4.25 (A14)
- net Z19: now also U4.4 (A1)
- net Z2: now also U4.2 (A3)
- net Z20: now also U4.30 (A9)
- net Z3: now also U4.3 (A2)
- net Z4: now also U4.28 (A11)
- net Z5: now also U4.29 (A10)
- net Z6: now also U4.5 (A0)
- net Z7: now also U4.20 (A19)
- net Z8: now also U4.21 (A18)
- net Z9: now also U4.22 (A17)
- net ~{CE}: now also U2.T12 (IO_L22P_T3_A05_D21_14), U4.7 (*CE); no longer U2.T14 (IO_L13P_T2_MRCC_14)
- net ~{WE}: now also U2.T14 (IO_L13P_T2_MRCC_14), U4.18 (*WE); no longer U2.T12 (IO_L22P_T3_A05_D21_14)
- net ~{Z0}: now also U4.43 (*UB)
Other:
- moved on the sheet: U8

Commit message: refine design
Parts:
- removed J8: RomAddr, Connector_PinHeader_2.54mm:PinHeader_1x08_P2.54mm_Vertical, symbol Connector_Generic:Conn_01x08
- added U6: SST39LF040-55, PCM_Package_LCC_AKL:PLCC-32_THT-Socket, symbol Memory_Flash:SST39SF040
Connections:
- net +3V3: now also U6.32 (VCC)
- net A0: now also U6.12 (A0)
- net A1: now also U6.11 (A1)
- net A10: now also U6.23 (A10)
- net A11: now also U6.25 (A11)
- net A12: now also U6.4 (A12)
- net A2: now also U6.10 (A2)
- net A3: now also U6.9 (A3)
- net A4: now also U6.8 (A4)
- net A5: now also U6.7 (A5)
- net A6: now also U6.6 (A6)
- net A7: now also U6.5 (A7)
- net A8: now also U6.27 (A8)
- net A9: now also U6.26 (A9)
- net GND: now also U6.16 (GND), U6.22 (CE); no longer J7.10 (Pin_10)
- net RD0: now also U6.13 (D0)
- net RD1: now also U6.14 (D1)
- net RD2: now also U6.15 (D2)
- net RD3: now also U6.17 (D3)
- net RD4: now also U6.18 (D4)
- net RD5: now also U6.19 (D5)
- net RD6: now also U6.20 (D6)
- net RD7: now also U6.21 (D7)
- net RZ13: now also U6.28 (A13)
- net RZ14: now also U2.H14 (IO_25_15), U6.29 (A14); no longer U2.H16 (IO_L20P_T3_A20_15)
- net RZ15: now also U6.3 (A15)
- net RZ16: now also U2.J18 (IO_L3P_T0_DQS_PUDC_B_14), U6.2 (A16); no longer U2.G14 (IO_L22P_T3_A17_15)
- net RZ17: now also U6.30 (A17)
- net RZ18: now also U2.K18 (IO_L3N_T0_DQS_EMCCLK_14), U6.1 (A18); no longer U2.H14 (IO_25_15)
- net ~{ROE}: now also U2.H16 (IO_L20P_T3_A20_15), U6.24 (OE); no longer U2.K18 (IO_L3N_T0_DQS_EMCCLK_14)
- net ~{RWE}: now also U2.G14 (IO_L22P_T3_A17_15), U6.31 (PGM); no longer U2.J18 (IO_L3P_T0_DQS_PUDC_B_14)
- net BUSY: now reaches U2.P14 (IO_L12P_T1_MRCC_14)
- net BUSY: now also J7.10 (Pin_10)
Other:
- moved on the sheet: R2, R3, R5, U4, U5

Commit message: complete primary routing
Parts:
- removed R1: 4.7K, PCM_Resistor_SMD_AKL:R_0402_1005Metric, symbol Device:R_Small
- removed U1: 74LVC573, Package_SO:TSSOP-20_4.4x6.5mm_P0.65mm, symbol 74xx:74LS373
- removed U2: XC7A15T-CSG325, Package_BGA:BGA-324_15x15mm_Layout18x18_P0.8mm, symbol FPGA_Xilinx_Artix7:XC7A15T-CSG325
- removed U9: AT28BV64B-20JU, Package_LCC:PLCC-32_THT-Socket, symbol Library:AT28BV64B-20JU
- added J8: AudioOut, Connector_PinHeader_2.54mm:PinHeader_1x08_P2.54mm_Vertical, symbol Connector_Generic:Conn_01x08
- added R8: 4.7K, PCM_Resistor_SMD_AKL:R_0402_1005Metric, symbol Device:R_Small
- added U7: XC7A35T-CSG324, Package_BGA:BGA-324_15x15mm_Layout18x18_P0.8mm, symbol FPGA_Xilinx_Artix7:XC7A35T-CSG324
Connections:
- net +1V0: now also U7.F10 (VCCBRAM), U7.F8 (VCCINT), U7.G11 (VCCBRAM), U7.G7 (VCCINT), U7.G9 (VCCINT), U7.H8 (VCCINT), U7.J11 (VCCINT), U7.J7 (VCCINT), U7.K8 (VCCINT), U7.L11 (VCCINT), U7.L7 (VCCINT), U7.M10 (VCCINT), U7.M8 (VCCINT), U7.N11 (VCCINT), U7.N7 (VCCINT), U7.N9 (VCCINT)
- net +1V8: now also U7.E8 (VCCBATT_0), U7.F12 (VCCAUX), U7.H10 (VCCADC_0), U7.H12 (VCCAUX), U7.K12 (VCCAUX), U7.M12 (VCCAUX)
- net +3V3: now also R8.2, U7.A17 (VCCO_15), U7.A7 (VCCO_35), U7.B10 (VCCO_16), U7.C13 (VCCO_15), U7.C3 (VCCO_35), U7.D16 (VCCO_15), U7.D6 (VCCO_35), U7.F2 (VCCO_35), U7.G15 (VCCO_15), U7.G5 (VCCO_35), U7.H18 (VCCO_15), U7.J1 (VCCO_35), U7.K14 (VCCO_15), U7.K4 (VCCO_34), U7.L17 (VCCO_14), U7.N13 (VCCO_14), U7.N3 (VCCO_34), U7.P12 (M0_0), U7.P16 (VCCO_14), U7.P6 (VCCO_34), U7.P8 (CFGBVS_0), U7.R9 (VCCO_0), U7.T12 (VCCO_14), U7.T2 (VCCO_34), U7.U15 (VCCO_14), U7.U5 (VCCO_34), U7.V18 (VCCO_14), U7.V8 (VCCO_34)
- net A0: now also U7.A11 (IO_L4N_T0_15)
- net A1: now also U7.B11 (IO_L4P_T0_15)
- net A10: now also U7.C14 (IO_L1N_T0_AD0N_15)
- net A11: now also U7.A15 (IO_L8P_T1_AD10P_15)
- net A12: now also U7.C15 (IO_L12N_T1_MRCC_15)
- net A13: now also U7.A16 (IO_L8N_T1_AD10N_15)
- net A14: now also U7.B16 (IO_L7P_T1_AD2P_15)
- net A15: now also U7.A18 (IO_L10N_T1_AD11N_15)
- net A2: now also U7.B12 (IO_L3N_T0_DQS_AD1N_15)
- net A3: now also U7.C12 (IO_L3P_T0_DQS_AD1P_15)
- net A4: now also U7.D12 (IO_L6P_T0_15)
- net A5: now also U7.A13 (IO_L9P_T1_DQS_AD3P_15)
- net A6: now also U7.B13 (IO_L2P_T0_AD8P_15)
- net A7: now also U7.D13 (IO_L6N_T0_VREF_15)
- net A8: now also U7.A14 (IO_L9N_T1_DQS_AD3N_15)
- net A9: now also U7.B14 (IO_L2N_T0_AD8N_15)
- net AVMA: now also U7.U14 (IO_L22P_T3_A05_D21_14)
- net B0: now also U7.E2 (IO_L14P_T2_SRCC_35)
- net B1: now also U7.E1 (IO_L18N_T2_35)
- net B2: now also U7.E3 (IO_L12P_T1_MRCC_35)
- net B3: now also U7.D2 (IO_L14N_T2_SRCC_35)
- net BA: now also U7.T16 (IO_L15N_T2_DQS_DOUT_CSO_B_14)
- net BS: now also U7.U16 (IO_L18P_T2_A12_D28_14)
- net BUSY: now also U7.T14 (IO_L14P_T2_SRCC_14)
- net CLKx2: now also U7.N5 (IO_L13P_T2_MRCC_34)
- net CSS: now also U7.C16 (IO_L20P_T3_A20_15)
- net E: now also U7.F16 (IO_L14N_T2_SRCC_15)
- net FPGA_CCLK: now also U7.E9 (CCLK_0)
- net FPGA_CSO_B: now also U7.L13 (IO_L6P_T0_FCS_B_14)
- net FPGA_DONE: now also U7.P10 (DONE_0)
- net FPGA_DQ0: now also U7.K17 (IO_L1P_T0_D00_MOSI_14)
- net FPGA_DQ1: now also U7.K18 (IO_L1N_T0_D01_DIN_14)
- net FPGA_DQ2: now also U7.L14 (IO_L2P_T0_D02_14)
- net FPGA_DQ3: now also U7.M14 (IO_L2N_T0_D03_14)
- net Format: now also U7.C4 (IO_L7P_T1_AD6P_35)
- net G0: now also U7.B3 (IO_L10P_T1_AD15P_35)
- net G1: now also U7.A3 (IO_L8N_T1_AD14N_35)
- net G2: now also U7.B2 (IO_L10N_T1_AD15N_35)
- net G3: now also U7.A1 (IO_L9N_T1_DQS_AD7N_35)
- net GM0: now also U7.D15 (IO_L12P_T1_MRCC_15)
- net GM1: now also U7.D17 (IO_L16N_T2_A27_15)
- net GM2: now also U7.D18 (IO_L21N_T3_DQS_A18_15)
- net GND: now also J8.2 (Pin_2), J8.4 (Pin_4), J8.6 (Pin_6), J8.8 (Pin_8), U7.A12 (GND), U7.A2 (GND), U7.B15 (GND), U7.B5 (GND), U7.C18 (GND), U7.C8 (GND), U7.D1 (GND), U7.D11 (GND), U7.E14 (GND), U7.E4 (GND), U7.F11 (GND), U7.F17 (GND), U7.F7 (GND), U7.F9 (GND), U7.G10 (GND), U7.G12 (GND), U7.G8 (GND), U7.H11 (GND), U7.H13 (GND), U7.H3 (GND), U7.H7 (GND), U7.H9 (GNDADC_0), U7.J10 (VP_0), U7.J12 (GND), U7.J16 (GND), U7.J6 (GND), U7.J8 (GND), U7.J9 (VREFN_0), U7.K10 (VREFP_0), U7.K11 (GND), U7.K7 (GND), U7.K9 (VN_0), U7.L10 (DXP_0), U7.L12 (GND), U7.L2 (GND), U7.L8 (GND), U7.L9 (DXN_0), U7.M11 (GND), U7.M15 (GND), U7.M5 (GND), U7.M7 (GND), U7.M9 (GND), U7.N10 (GND), U7.N12 (GND), U7.N18 (GND), U7.N8 (GND), U7.P1 (GND), U7.P11 (M2_0), U7.P13 (M1_0), U7.R14 (GND), U7.R4 (GND), U7.T17 (GND), U7.T7 (GND), U7.U10 (GND), U7.V13 (GND), U7.V3 (GND)
- net HALT: now also U7.V15 (IO_L16P_T2_CSI_B_14)
- net LIC: now also U7.V14 (IO_L22N_T3_A04_D20_14)
- net PROG_B: now also U7.P9 (PROGRAM_B_0)
- net Q: now also U7.F18 (IO_L22N_T3_A16_15)
- net R0: now also U7.D3 (IO_L12N_T1_MRCC_35)
- net R1: now also U7.D4 (IO_L11N_T1_SRCC_35)
- net R2: now also U7.C1 (IO_L16N_T2_35)
- net R3: now also U7.C2 (IO_L16P_T2_35)
- net RD0: now also U7.T1 (IO_L17N_T2_34)
- net RD1: now also U7.T3 (IO_L11N_T1_SRCC_34)
- net RD2: now also U7.U1 (IO_L7P_T1_34)
- net RD3: now also U7.U2 (IO_L9P_T1_DQS_34)
- net RD4: now also U7.V1 (IO_L7N_T1_34)
- net RD5: now also U7.V2 (IO_L9N_T1_DQS_34)
- net RD6: now also U7.U3 (IO_L8N_T1_34)
- net RD7: now also U7.V4 (IO_L10N_T1_34)
- net RZ13: now also U7.L3 (IO_L2N_T0_34)
- net RZ14: now also U7.K1 (IO_L23N_T3_35)
- net RZ15: now also U7.K2 (IO_L23P_T3_35)
- net RZ16: now also U7.L4 (IO_L5N_T0_34)
- net RZ17: now also U7.K3 (IO_L2P_T0_34)
- net RZ18: now also U7.M2 (IO_L4N_T0_34)
- net R/~{W}: now also U7.B17 (IO_L7N_T1_AD2N_15)
- net S0: now also U7.G16 (IO_L13N_T2_MRCC_15)
- net S1: now also U7.G17 (IO_L18N_T2_A23_15)
- net S2: now also U7.G18 (IO_L22P_T3_A17_15)
- net TCK: now also U7.E10 (TCK_0)
- net TDI: now also U7.E11 (TDI_0)
- net TDO: now also U7.E13 (TDO_0)
- net TMS: now also U7.E12 (TMS_0)
- net TSC: now also U7.T15 (IO_L14N_T2_SRCC_14)
- net VCLK: now also U7.B1 (IO_L9P_T1_DQS_AD7P_35)
- net Z0: now also U7.U6 (IO_L22N_T3_34)
- net Z1: now also U7.U4 (IO_L8P_T1_34)
- net Z10: now also U7.T9 (IO_L24P_T3_A01_D17_14)
- net Z11: now also U7.U9 (IO_L21P_T3_DQS_34)
- net Z12: now also U7.V9 (IO_L21N_T3_DQS_34)
- net Z13: now also U7.T10 (IO_L24N_T3_A00_D16_14)
- net Z14: now also U7.V10 (IO_L21P_T3_DQS_14)
- net Z15: now also U7.T11 (IO_L19P_T3_A10_D26_14)
- net Z16: now also U7.V12 (IO_L20N_T3_A07_D23_14)
- net Z17: now also U7.T13 (IO_L23P_T3_A03_D19_14)
- net Z18: now also U7.U13 (IO_L23N_T3_A02_D18_14)
- net Z19: now also U7.V6 (IO_L20N_T3_34)
- net Z2: now also U7.V5 (IO_L10P_T1_34)
- net Z20: now also U7.U11 (IO_L19N_T3_A09_D25_VREF_14)
- net Z3: now also U7.T5 (IO_L12P_T1_MRCC_34)
- net Z4: now also U7.U12 (IO_L20P_T3_A08_D24_14)
- net Z5: now also U7.V11 (IO_L21N_T3_DQS_A06_D22_14)
- net Z6: now also U7.U7 (IO_L22P_T3_34)
- net Z7: now also U7.V7 (IO_L20P_T3_34)
- net Z8: now also U7.T8 (IO_L24N_T3_34)
- net Z9: now also U7.U8 (IO_25_34)
- net ~{A}/G: now also U7.B18 (IO_L10P_T1_AD11P_15)
- net ~{CE}: now also U7.R6 (IO_L19P_T3_34)
- net ~{FIRQ}: now also U7.U17 (IO_L17P_T2_A14_D30_14)
- net ~{FS}: now also U7.E17 (IO_L16P_T2_A28_15)
- net ~{HS}: now also U7.E18 (IO_L21P_T3_DQS_15)
- net ~{IRQ}: now also U7.V16 (IO_L16N_T2_A15_D31_14)
- net ~{NMI}: now also U7.V17 (IO_L18N_T2_A11_D27_14)
- net ~{ROE}: now also U7.M1 (IO_L1N_T0_34)
- net ~{RST}: now also U7.C17 (IO_L20N_T3_A19_15)
- net ~{RWE}: now also U7.L1 (IO_L1P_T0_34)
- net ~{WE}: now also U7.R8 (IO_L24P_T3_34)
- net ~{Z0}: now also U7.T6 (IO_L23N_T3_34)
- new net: R8.1, U7.P7 (INIT_B_0)
- new net BCLK: J8.1 (Pin_1), U7.F3 (IO_L13N_T2_MRCC_35)
- new net MCLK: J8.7 (Pin_7), U7.G4 (IO_L20P_T3_35)
- new net SD: J8.5 (Pin_5), U7.G1 (IO_L17N_T2_35)
- new net WS: J8.3 (Pin_3), U7.F1 (IO_L18P_T2_35)
- no-connect marks 21 -> 110
Other:
- moved on the sheet: C1, C10, C11, C2, C25, C3, C4, C49, C5, C50, C6, C7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
